File: vectron_vga_plus_design/vectron_vga_plus_design.sch (KiCad schematic (older format))
At the start: 19 parts

Commit message: Save progress on design files.
Parts:
- added J?: Conn_02x01, symbol Connector_Generic:Conn_02x01
Connections:
- net +5V: now also U?.14 (VCC), U?.14 (VCC), U?.20 (VCC), U?.20 (VCC), U?.20 (VCC)
- net GND: now also U?.1 (A18), U?.1 (DIR), U?.1 (DIR), U?.10 (GND), U?.10 (GND), U?.10 (GND), U?.7 (GND), U?.7 (GND)
- net at U?.11 (P4), U?.11 (Q3): now also U?.15 (B4)
- net at U?.12 (Q2), U?.13 (P5): now also U?.16 (B3)
- net at U?.13 (Q1), U?.15 (P6): now also U?.17 (B2)
- net at U?.14 (Q0), U?.17 (P7): now also U?.18 (B1)
- net at U?.11 (Q3), U?.2 (P0): now also U?.11 (B8)
- net at U?.12 (Q2), U?.4 (P1): now also U?.12 (B7)
- net at U?.13 (Q1), U?.6 (P2): now also U?.13 (B6)
- net at U?.14 (Q0), U?.8 (P3): now also U?.14 (B5)
- net at U?.19 (*P=Q): now also U?.13 (4B)
- net at U?.1 (1A): now also U?.8 (3Y)
- net at U?.10 (3B): now also U?.11 (4Y)
- net at U?.2 (1B): now also U?.12 (6Y)
- net at U?.9 (3A): now also U?.10 (5Y)
- net at U?.1 (1A): now also U?.19 (2~G/2G+), U?.29 (WE), J?.1 (Pin_1)
- net at U?.2 (1Y): now also U?.19 (2~G/2G+), U?.19 (~OE), U?.19 (~OE), U?.24 (OE)
- net at U?.3 (2A): now also U?.22 (CE), J?.2 (Pin_2)
- net at U?.2 (A1): now also U?.12 (A0)
- net at U?.3 (A2): now also U?.11 (A1)
- net at U?.4 (A3): now also U?.10 (A2)
- net at U?.5 (A4): now also U?.9 (A3)
- net at U?.6 (A5): now also U?.8 (A4)
- net at U?.7 (A6): now also U?.7 (A5)
- net at U?.8 (A7): now also U?.6 (A6)
- net at U?.9 (A8): now also U?.5 (A7)
- net at U?.2 (A1): now also U?.27 (A8)
- net at U?.3 (A2): now also U?.26 (A9)
- net at U?.4 (A3): now also U?.23 (A10)
- net at U?.5 (A4): now also U?.25 (A11)
- net at U?.6 (A5): now also U?.4 (A12)
- net at U?.7 (A6): now also U?.28 (A13)
- net at U?.8 (A7): now also U?.3 (A14)
- net at U?.9 (A8): now also U?.31 (A15)

Commit message: Save progress on design files.
Parts:
- added J?: Address Bus, symbol Connector:Conn_01x18_Male
- added J?: Data Bus, symbol Connector:Conn_01x05_Male
- added J?: VGA, symbol Connector:Conn_01x05_Male
- added J?: Power, symbol Connector:Conn_01x05_Male
- added R? (x3): 200 ohm, symbol Device:R
- added R? (x3): 100 ohm, symbol Device:R
Connections:
- net +5V: now also U?.1 (~Mr), U?.20 (VCC), U?.20 (VCC), U?.20 (VCC), U?.20 (VCC), U?.20 (VCC)
- net GND: now also U?.10 (GND), U?.10 (GND), U?.10 (GND), U?.10 (GND), U?.10 (GND), R?.2, R?.2, R?.2
- net at U?.11 (P4), U?.11 (Q3): now also U?.15 (B4)
- net at U?.12 (Q2), U?.13 (P5): now also U?.16 (B3)
- net at U?.13 (Q1), U?.15 (P6): now also U?.17 (B2)
- net at U?.14 (Q0), U?.17 (P7): now also U?.18 (B1)
- net at U?.11 (Q3), U?.2 (P0): now also U?.11 (B8)
- net at U?.12 (Q2), U?.4 (P1): now also U?.12 (B7)
- net at U?.13 (Q1), U?.6 (P2): now also U?.13 (B6)
- net at U?.14 (Q0), U?.8 (P3): now also U?.14 (B5)
- net at U?.2 (Q0): now also R?.1
- net at U?.3 (D0): now also U?.7 (2Y2)
- net at U?.4 (D1): now also U?.5 (2Y3)
- net at U?.5 (Q1): now also R?.1
- net at U?.6 (Q2): now also R?.1
- net at U?.7 (D2): now also U?.3 (2Y4)
- net at J?.1 (Pin_1), U?.1 (1A), U?.19 (2~G/2G+)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: now also U?.1 (1~G), U?.1 (1~G), U?.1 (1~G), U?.19 (2~G/2G+), U?.19 (2~G/2G+)
- net at U?.19 (2~G/2G+), U?.19 (~OE), U?.19 (~OE)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: now also U?.1 (1~G)
- net at U?.12 (A0), U?.2 (A1): now also U?.18 (1Y1)
- net at U?.11 (A1), U?.3 (A2): now also U?.16 (1Y2)
- net at U?.10 (A2), U?.4 (A3): now also U?.14 (1Y3)
- net at U?.5 (A4), U?.9 (A3): now also U?.12 (1Y4)
- net at U?.6 (A5), U?.8 (A4): now also U?.9 (2Y1)
- net at U?.7 (A5), U?.7 (A6): now also U?.7 (2Y2)
- net at U?.6 (A6), U?.8 (A7): now also U?.5 (2Y3)
- net at U?.5 (A7), U?.9 (A8): now also U?.3 (2Y4)
- net at U?.2 (A1), U?.27 (A8): now also U?.18 (1Y1)
- net at U?.26 (A9), U?.3 (A2): now also U?.16 (1Y2)
- net at U?.23 (A10), U?.4 (A3): now also U?.14 (1Y3)
- net at U?.25 (A11), U?.5 (A4): now also U?.12 (1Y4)
- net at U?.4 (A12), U?.6 (A5): now also U?.9 (2Y1)
- net at U?.28 (A13), U?.7 (A6): now also U?.7 (2Y2)
- net at U?.3 (A14), U?.8 (A7): now also U?.5 (2Y3)
- net at U?.31 (A15), U?.9 (A8): now also U?.3 (2Y4)
- net at U?.11 (2A1): now also J?.5 (Pin_5)
- net at U?.13 (2A2): now also J?.6 (Pin_6)
- net at U?.15 (2A3): now also J?.7 (Pin_7)
- net at U?.17 (2A4): now also J?.8 (Pin_8)
- net at U?.2 (1A1): now also J?.1 (Pin_1)
- net at U?.4 (1A2): now also J?.2 (Pin_2)
- net at U?.6 (1A3): now also J?.3 (Pin_3)
- net at U?.8 (1A4): now also J?.4 (Pin_4)
- net at U?.11 (2A1): now also J?.13 (Pin_13)
- net at U?.13 (2A2): now also J?.14 (Pin_14)
- net at U?.15 (2A3): now also J?.15 (Pin_15)
- net at U?.17 (2A4): now also J?.16 (Pin_16)
- net at U?.2 (1A1): now also J?.9 (Pin_9)
- net at U?.4 (1A2): now also J?.10 (Pin_10)
- net at U?.6 (1A3): now also J?.11 (Pin_11)
- net at U?.8 (1A4): now also J?.12 (Pin_12)
- net at U?.11 (2A1): now also J?.4 (Pin_4)
- net at U?.12 (1Y4): now also U?.15 (DQ2), U?.17 (2A4)
- net at U?.13 (2A2): now also J?.5 (Pin_5)
- net at U?.14 (1Y3): now also U?.14 (DQ1), U?.15 (2A3)
- net at U?.16 (1Y2): now also U?.13 (2A2), U?.13 (DQ0)
- net at U?.17 (2A4): now also J?.18 (Pin_18)
- net at U?.18 (1Y1): now also U?.2 (A16), U?.9 (2Y1)
- net at U?.2 (1A1): now also J?.17 (Pin_17)
- net at U?.3 (2Y4): now also U?.12 (1Y4), U?.30 (A17)
- net at U?.4 (1A2): now also J?.1 (Pin_1)
- net at U?.6 (1A3): now also J?.2 (Pin_2)
- net at U?.7 (2Y2): now also U?.18 (DQ4)
- net at U?.8 (1A4): now also J?.3 (Pin_3)
- net at U?.9 (2Y1): now also U?.17 (DQ3)
- new net: J?.1 (Pin_1), R?.1, R?.2
- new net: J?.2 (Pin_2), R?.1, R?.2
- new net: J?.3 (Pin_3), R?.1, R?.2

Commit message: Save progress on design files.
Parts:
- added C? (x4): 220 uF, symbol Device:CP1
- added J?: G, symbol Connector:Conn_01x01_Male
- added J?: L77HDE15SD1CH4F, AMPHENOL_L77HDE15SD1CH4F, symbol L77HDE15SD1CH4F:L77HDE15SD1CH4F
- J?: value Address Bus -> Address In
- J?: value Data Bus -> Data In
- J?: value VGA -> VGA Out
Connections:
- net +5V: now also J?.1 (Pin_1), J?.2 (Pin_2), U?.32 (VCC), C?.1, C?.1, C?.1, C?.1
- net B: now also J?.3 (Pin_3), R?.1, R?.2, J?.3
- net G: now also J?.2 (Pin_2), R?.1, R?.2, J?.2
- net GND: now also J?.3 (Pin_3), J?.4 (Pin_4), J?.5 (Pin_5), U?.16 (VSS), C?.2, C?.2, C?.2, C?.2, J?.1 (Pin_1), J?.10, J?.5, J?.6, J?.7, J?.8
- net at U?.18 (D7): now also U?.18 (DQ4), U?.7 (2Y2)
- net at U?.19 (Q7): now also J?.5 (Pin_5), J?.14
- net at U?.8 (D3): now also U?.17 (DQ3), U?.18 (1Y1), U?.2 (A16), U?.9 (2Y1), U?.9 (2Y1)
- net at U?.9 (Q3): now also J?.4 (Pin_4), J?.13
- net at J?.1 (Pin_1), R?.1, R?.2: now also J?.1
- new net: J?.S1 (SHIELD), J?.S2 (SHIELD)
Other:
- moved on the sheet: J?

Commit message: Save progress on design files.
Parts:
- C1, C2, C3, C4: renamed from C?; footprint (none) -> Capacitor_THT:CP_Radial_D10.0mm_P7.50mm
- J1: renamed from J?; footprint (none) -> Connector_PinHeader_2.54mm:PinHeader_1x18_P2.54mm_Horizontal
- J2, J4, J5: renamed from J?; footprint (none) -> Connector_PinHeader_2.54mm:PinHeader_1x05_P2.54mm_Horizontal
- J3: renamed from J?; footprint (none) -> Connector_PinHeader_2.54mm:PinHeader_1x01_P2.54mm_Horizontal
- J6: renamed from J?; footprint AMPHENOL_L77HDE15SD1CH4F -> L77HDE15SD1CH4F:AMPHENOL_L77HDE15SD1CH4F
- J7: renamed from J?; footprint (none) -> Connector_PinHeader_2.54mm:PinHeader_1x02_P2.54mm_Horizontal
- R1, R2, R3, R4, R5, R6: renamed from R?; footprint (none) -> Resistor_THT:R_Axial_DIN0207_L6.3mm_D2.5mm_P7.62mm_Horizontal
- U1, U6: renamed from U?; footprint N20 -> 74ls682:SN74LS682N
- U10: renamed from U?; footprint DIP794W45P254L1969H508Q14 -> SN74HC32N:DIP794W45P254L1969H508Q14
- U11, U14, U18, U7, U8: renamed from U?; footprint (none) -> footprints:SN74LS161AN
- U12: renamed from U?; footprint DIP254P1524X393-32 -> AS6C4008-55PCN:DIP254P1524X393-32
- U13: renamed from U?; footprint DIP794W45P254L1969H508Q14 -> SN74LS04N:DIP794W45P254L1969H508Q14
- U15, U17: renamed from U?; footprint DIP254P762X508-20 -> SN74LS245N:DIP254P762X508-20
- U16, U2, U5, U9: renamed from U?; footprint DIP254P762X508-20 -> SN74LS244N:DIP254P762X508-20
- U3: renamed from U?; footprint (none) -> SN74LS244N:DIP254P762X508-20
- U4: renamed from U?; footprint DIP794W45P254L1969H508Q14 -> SN74LS74AN:DIP794W45P254L1969H508Q14
- gave numbers to parts that had none: 1
Connections:
- net at U12.17 (DQ3), U3.8 (D3), U9.9 (2Y1): no longer U12.2 (A16), U16.9 (2Y1), U9.18 (1Y1)
- new net: U12.2 (A16), U16.9 (2Y1), U9.18 (1Y1)

Commit message: Save progress on design files.
Connections:
- net at J7.2 (Pin_2), U12.22 (CE): no longer U13.3 (2A)
Changed lines of the file:
@@
 Connection ~ 11300 4200
-Wire Wire Line
-	9600 4300 9400 4300
-Wire Wire Line
-	9400 4300 9400 6750
 Wire Wire Line
 	9400 7550 9450 7550
@@
 Wire Wire Line
 	17950 6750 17950 7700
-Connection ~ 9400 6750
 Wire Wire Line
 	9400 6750 9400 7550

Commit message: Save progress on design files.
Parts:
- J7: value Conn_02x01 -> Mode
Changed lines of the file:
@@
 P 17650 7700
 F 0 "J7" H 17700 7917 50  0000 C CNN
-F 1 "Conn_02x01" H 17700 7826 50  0000 C CNN
+F 1 "Mode" H 17700 7826 50  0000 C CNN
 F 2 "Connector_PinHeader_2.54mm:PinHeader_1x02_P2.54mm_Horizontal" H 17650 7700 50  0001 C CNN
 F 3 "~" H 17650 7700 50  0001 C CNN
