File: vectron_vga_plus_design/vectron_vga_plus_design.kicad_pcb (KiCad board)
At the start: 4 copper layers, 177.8 x 139.7 mm, 36 parts, among them J1 Address In, J2 Data In, J3 G, J4 VGA Out, J5 Power, J6 L77HDE15SD1CH4F, J7 Mode, U1 SN74LS682N, U10 SN74HC32N, U11 74LS161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

Commit message: Save progress on design files.
Parts:
- moved U3 142.4 mm to (560.1, 569.0), turned to 90 degrees
- moved U17 21.7 mm to (560.1, 508.0), turned to 90 degrees
- moved R6 7.62 mm to (525.8, 593.1), turned to 90 degrees
- moved U16 1.80 mm to (537.2, 552.5)
Routing:
- net Net-(J7-Pad1): track 0.00 -> 171.4 mm
- net Net-(U13-Pad13): track 0.00 -> 152.6 mm, vias 0 -> 5
- net Net-(J2-Pad1): track 0.00 -> 111.8 mm
- net Net-(J1-Pad1): track 0.00 -> 108.7 mm
- net Net-(J1-Pad17): track 0.00 -> 105.3 mm
- net Net-(U11-Pad2): track 120.9 -> 225.5 mm
- net Net-(J1-Pad18): track 0.00 -> 103.7 mm
- net Net-(U12-Pad17): track 0.00 -> 99.9 mm
- net Net-(J2-Pad2): track 0.00 -> 99.7 mm
- net Net-(J1-Pad16): track 0.00 -> 96.2 mm
- net Net-(J1-Pad2): track 0.00 -> 94.4 mm
- net Net-(J1-Pad3): track 0.00 -> 93.4 mm
- net Net-(J1-Pad9): track 0.00 -> 93.2 mm
- net Net-(J1-Pad10): track 0.00 -> 91.4 mm
- net Net-(J2-Pad3): track 0.00 -> 91.3 mm
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Other:
- board text added: "A0"
- board text added: "B"
- board text added: "CE"
- board text added: "D0"
- board text added: "GND"
- board text added: "H"
- board text added: "R"
- board text added: "V"
- board text added: "WE"

Commit message: Save progress on design files.
Routing:
- net Net-(U12-Pad6): track 35.4 -> 308.7 mm, vias 0 -> 2
- net Net-(U1-Pad4): track 52.3 -> 281.6 mm, vias 1 -> 2
- net Net-(U12-Pad31): track 64.3 -> 281.6 mm, vias 0 -> 1
- net Net-(U12-Pad5): track 35.4 -> 215.0 mm, vias 0 -> 1
- net Net-(U1-Pad2): track 75.5 -> 231.4 mm, vias 0 -> 1
- net Net-(U1-Pad17): track 40.0 -> 193.3 mm, vias 0 -> 1
- net Net-(U10-Pad3): track 91.1 -> 242.7 mm, vias 0 -> 1
- net Net-(U12-Pad8): track 35.4 -> 181.3 mm, vias 0 -> 5
- net Net-(U14-Pad13): track 43.4 -> 186.7 mm, vias 1 -> 5
- net Net-(U11-Pad14): track 45.1 -> 184.6 mm, vias 1 -> 3
- net Net-(U14-Pad14): track 39.9 -> 178.6 mm, vias 2 -> 4
- net Net-(U12-Pad30): track 0.00 -> 109.7 mm, vias 0 -> 3
- net Net-(U12-Pad7): track 35.4 -> 145.0 mm
- net Net-(U12-Pad15): track 0.00 -> 105.4 mm, vias 0 -> 3
- net Net-(U1-Pad13): track 53.7 -> 152.1 mm
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
Commit message: Save progress on design files.
Routing:
- net Net-(U12-Pad7): track 145.0 -> 431.4 mm, vias 0 -> 5
- net Net-(U12-Pad13): track 26.0 -> 298.4 mm, vias 1 -> 3
- net Net-(J7-Pad1): track 171.4 -> 391.9 mm, vias 0 -> 3
- net Net-(U12-Pad25): track 68.4 -> 282.3 mm, vias 2 -> 6
- net Net-(U12-Pad11): track 35.4 -> 193.4 mm, vias 0 -> 3
- net Net-(U12-Pad28): track 65.8 -> 216.3 mm, vias 0 -> 5
- net Net-(U12-Pad31): track 281.6 -> 425.4 mm, vias 1 -> 3
- net Net-(U12-Pad3): track 57.9 -> 198.6 mm, vias 0 -> 1
- net Net-(U12-Pad10): track 35.4 -> 164.6 mm, vias 0 -> 2
- net Net-(U12-Pad12): track 35.4 -> 161.5 mm, vias 0 -> 3
- net Net-(U12-Pad26): track 60.8 -> 164.6 mm, vias 2 -> 5
- net Net-(U12-Pad4): track 55.4 -> 154.3 mm
- net Net-(U12-Pad24): track 120.2 -> 207.1 mm, vias 1 -> 2
- net Net-(U12-Pad14): track 21.4 -> 96.4 mm, vias 1 -> 3
- net Net-(U12-Pad23): track 72.5 -> 138.8 mm, vias 0 -> 3
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Other:
- board text added: "74LS244N"
- board text added: "74LS245N"
- board text added: "74LS74AN"
- board text added: "Address In"
- board text added: "Data In"
- board text added: "Hs"
- board text added: "Mode"
- board text added: "Nick Bild November 2021 github.com/nickbild/vectron_vga_plus"
- board text added: "Power"
- board text added: "VGA Out"
- board text added: "Vectron VGA Plus"
- board text added: "Vs"
- board text removed: "H"
- board text removed: "V"
